File: Dragon64Board/dragon64.kicad_pcb (KiCad board)
At the start: 2 copper layers, 333.2 x 229.3 mm, 234 parts, among them IC1 74LS244, IC10 6847, IC11 6551, IC12 74LS393, IC13 74LS32, IC14 74LS74, IC15 4164, IC16 4164, IC17 LM1889N, IC18 74LS86, IC19 74LS00, IC2 LM393, IC20 74LS273, IC21 4164, IC22 4164, IC23 74LS393, IC24 74LS390, IC25 74LS244, IC26 4164, IC27 4164, IC28 LM318N, IC29 4053, IC30 74LS74, IC31 74LS123, IC32 4164, IC33 4164, IC34 27C128, IC35 74LS00, IC36 74LS02, IC37 27C128, IC38 MC6809E, IC39 6883, IC4 4050, IC40 74LS138, IC5 6821, IC6 4529, IC7 4069, IC8 6821, IC9 74LS20, J1 ATX, J2 TTL Serial Connector, U1 MAX232, Y1 14.31818Mhz, Y2 1.8432Mhz, Y3 4.433619Mhz

Commit message: PAL to NTSC
Parts:
- removed C48: .01u, Capacitor_THT:C_Disc_D7.5mm_W2.5mm_P5.00mm
- removed C49: 4p7, Capacitor_THT:C_Disc_D7.5mm_W2.5mm_P5.00mm
- removed C54: 330p, Capacitor_THT:C_Disc_D7.5mm_W2.5mm_P5.00mm
- removed D21, D22: 1N4148, Diode_THT:D_DO-35_SOD27_P7.62mm_Horizontal
- removed IC12, IC23: 74LS393, Package_DIP:DIP-14_W7.62mm_Socket_LongPads
- removed IC13: 74LS32, Package_DIP:DIP-14_W7.62mm_Socket_LongPads
- removed IC14, IC30: 74LS74, Package_DIP:DIP-14_W7.62mm_Socket_LongPads
- removed IC17: LM1889N, Package_DIP:DIP-18_W7.62mm_Socket_LongPads
- removed IC18: 74LS86, Package_DIP:DIP-14_W7.62mm_Socket_LongPads
- removed IC19: 74LS00, Package_DIP:DIP-14_W7.62mm_Socket_LongPads
- removed IC24: 74LS390, Package_DIP:DIP-16_W7.62mm_Socket_LongPads
- removed IC28: LM318N, Package_DIP:DIP-8_W7.62mm_Socket_LongPads
- removed IC29: 4053, Package_DIP:DIP-16_W7.62mm_Socket_LongPads
- removed IC31: 74LS123, Package_DIP:DIP-16_W7.62mm_Socket_LongPads
- removed IC9: 74LS20, Package_DIP:DIP-14_W7.62mm_Socket_LongPads
- removed LK2: ~, Connector_PinHeader_2.54mm:PinHeader_1x03_P2.54mm_Vertical
- removed R42: 5K6, Resistor_THT:R_Axial_DIN0207_L6.3mm_D2.5mm_P7.62mm_Horizontal
- removed R43: 10R, Resistor_THT:R_Axial_DIN0207_L6.3mm_D2.5mm_P7.62mm_Horizontal
- removed R44: 680R, Resistor_THT:R_Axial_DIN0207_L6.3mm_D2.5mm_P7.62mm_Horizontal
- removed R45, R50, R51: 1K, Resistor_THT:R_Axial_DIN0207_L6.3mm_D2.5mm_P7.62mm_Horizontal
- removed R46: 270R, Resistor_THT:R_Axial_DIN0207_L6.3mm_D2.5mm_P7.62mm_Horizontal
- removed R47: 470R, Resistor_THT:R_Axial_DIN0207_L6.3mm_D2.5mm_P7.62mm_Horizontal
- removed R48: 220R, Resistor_THT:R_Axial_DIN0207_L6.3mm_D2.5mm_P7.62mm_Horizontal
- removed R49: 330R, Resistor_THT:R_Axial_DIN0207_L6.3mm_D2.5mm_P7.62mm_Horizontal
- removed R52, R57: 3K3, Resistor_THT:R_Axial_DIN0207_L6.3mm_D2.5mm_P7.62mm_Horizontal
- removed R53, R56: 2K7, Resistor_THT:R_Axial_DIN0207_L6.3mm_D2.5mm_P7.62mm_Horizontal
- removed R54, R55: 10K, Resistor_THT:R_Axial_DIN0207_L6.3mm_D2.5mm_P7.62mm_Horizontal
- removed R58: 1K2, Resistor_THT:R_Axial_DIN0207_L6.3mm_D2.5mm_P7.62mm_Horizontal
- removed R59: 6K8, Resistor_THT:R_Axial_DIN0207_L6.3mm_D2.5mm_P7.62mm_Horizontal
- removed R60: 15K, Resistor_THT:R_Axial_DIN0207_L6.3mm_D2.5mm_P7.62mm_Horizontal
- removed R61: 1K8, Resistor_THT:R_Axial_DIN0207_L6.3mm_D2.5mm_P7.62mm_Horizontal
- removed R62: 8K2, Resistor_THT:R_Axial_DIN0207_L6.3mm_D2.5mm_P7.62mm_Horizontal
- removed R63: 12K, Resistor_THT:R_Axial_DIN0207_L6.3mm_D2.5mm_P7.62mm_Horizontal
- removed R72: 22K, Resistor_THT:R_Axial_DIN0207_L6.3mm_D2.5mm_P7.62mm_Horizontal
- removed TR2, TR3: 2N2369A, Package_TO_SOT_THT:TO-18-3
- removed TR4: BC212L, Package_TO_SOT_THT:TO-92
- removed VR1: 10k, Potentiometer_THT:Potentiometer_Vishay_T7-YA_Single_Vertical
- removed Y3: 4.433619Mhz, Crystal:Crystal_HC49-U_Vertical
- added D4: 1N4002, Diode_THT:D_DO-35_SOD27_P7.62mm_Horizontal, F.Cu at (80.1, -6.10)
- added D5: 1N4148, Diode_THT:D_DO-35_SOD27_P7.62mm_Horizontal, F.Cu at (78.2, 52.1)
- added G***: LOGO, logo:we_small_neg, F.Cu at (220.3, 124.3)
- added J3: composite on luma, Connector_PinHeader_2.54mm:PinHeader_1x02_P2.54mm_Vertical, F.Cu at (13.4, -12.1)
- added Q1: BC557, Package_TO_SOT_THT:TO-92_Wide, F.Cu at (62.8, -5.11)
- added Q2: 2N2222, Package_TO_SOT_THT:TO-18-3, F.Cu at (64.3, 12.6)
- added Q3: 2N2222, Package_TO_SOT_THT:TO-18-3, F.Cu at (64.3, 3.73)
- added R11: 10K, Resistor_THT:R_Axial_DIN0207_L6.3mm_D2.5mm_P7.62mm_Horizontal, F.Cu at (48.0, 2.05)
- added R12: 390, Resistor_THT:R_Axial_DIN0207_L6.3mm_D2.5mm_P7.62mm_Horizontal, F.Cu at (36.7, -14.7)
- added R13: 820, Resistor_THT:R_Axial_DIN0207_L6.3mm_D2.5mm_P7.62mm_Horizontal, F.Cu at (48.0, -2.11)
- added R30: 420, Resistor_THT:R_Axial_DIN0207_L6.3mm_D2.5mm_P7.62mm_Horizontal, F.Cu at (48.0, -6.27)
- added R31: 470, Resistor_THT:R_Axial_DIN0207_L6.3mm_D2.5mm_P7.62mm_Horizontal, F.Cu at (55.6, 6.22)
- added R6: 470, Resistor_THT:R_Axial_DIN0207_L6.3mm_D2.5mm_P7.62mm_Horizontal, F.Cu at (55.6, 14.5)
- added R7: 390, Resistor_THT:R_Axial_DIN0207_L6.3mm_D2.5mm_P7.62mm_Horizontal, F.Cu at (80.0, -12.5)
- added R8: 5.6k, Resistor_THT:R_Axial_DIN0207_L6.3mm_D2.5mm_P7.62mm_Horizontal, F.Cu at (36.9, -10.9)
- added U2: MC1372, Package_DIP:DIP-14_W7.62mm_LongPads, F.Cu at (72.3, -1.24)
- C20: value 4.7uf tant -> .01u; footprint Capacitor_THT:CP_Radial_D4.0mm_P2.00mm -> Capacitor_THT:C_Disc_D7.5mm_W2.5mm_P5.00mm
- C21: value 3p3 -> .01u
- C29, C31: value 33p -> .01u
- C30: value .1u -> 56pf
- C32: value 2-22p -> .01u; footprint dragon64:C_Trimmer_D7.5mm -> Capacitor_THT:C_Disc_D7.5mm_W2.5mm_P5.00mm
- C33: value 4.7uf tant -> 0.1uf; footprint Capacitor_THT:CP_Radial_D4.0mm_P2.00mm -> Capacitor_THT:C_Disc_D7.5mm_W2.5mm_P5.00mm
- C35: value 180p -> 25uf
- C36: value 180p -> 100uf; footprint Capacitor_THT:C_Disc_D7.5mm_W2.5mm_P5.00mm -> Capacitor_THT:CP_Radial_D4.0mm_P2.00mm
- C37: value 180p -> 390pf
- C44: value 4.7uf tant -> 470pf; footprint Capacitor_THT:CP_Radial_D4.0mm_P2.00mm -> Capacitor_THT:C_Disc_D7.5mm_W2.5mm_P5.00mm
- H2: moved to B.Cu
- R41: value 1K2 -> 1K
- moved C19 225.9 mm to (194.1, -12.8)
- moved C18 195.0 mm to (224.7, 52.8)
- moved C12 193.5 mm to (197.0, 52.8)
- moved C28 180.2 mm to (251.8, 65.2), turned to 0 degrees
- moved C57 168.4 mm to (275.0, 24.2)
- moved IC8 164.7 mm to (219.3, 57.8)
- moved IC5 163.1 mm to (192.3, 57.8)
- moved C38 151.8 mm to (251.8, 24.2)
- moved C44 149.2 mm to (19.4, -16.1)
- moved C37 142.5 mm to (54.3, -11.8)
- moved IC1 140.5 mm to (91.0, 10.0)
- moved IC25 137.0 mm to (268.7, 29.7)
- moved IC20 134.7 mm to (250.5, 29.7)
- moved C60 134.0 mm to (92.4, 4.75)
- moved C56 132.0 mm to (293.1, 24.2)
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Connections:
- net /PIAs/~FS renamed FS
- net /VCLK renamed VCLK
- C20 pad 1: Net-(C20-Pad1) -> +5V
- C21 pad 1: Net-(C21-Pad1) -> +5V
- C21 pad 2: +5V -> GND
- C22 pad 1: Net-(C22-Pad1) -> +5V
- C22 pad 2: Net-(C22-Pad2) -> GND
- C29 pad 1: Net-(C29-Pad1) -> +5V
- C29 pad 2: Net-(C29-Pad2) -> GND
- C30 pad 1: Net-(C29-Pad1) -> VCLK1
- C30 pad 2: Net-(C30-Pad2) -> GND
- C31 pad 1: -5V -> +5V
- C31 pad 2: Net-(C31-Pad2) -> GND
- C32 pad 1: Net-(C32-Pad1) -> +5V
- C32 pad 2: -5V -> GND
- C33 pad 1: GND -> +5V
- C33 pad 2: -5V -> GND
- C35 pad 1: GND -> +5V
- C35 pad 2: Net-(C35-Pad2) -> GND
- C36 pad 1: GND -> /Video/Y
- C37 pad 1: GND -> +5V
- C44 pad 1: +5V -> Net-(C44-Pad1)
- C44 pad 2: GND -> CHROMA
- IC10 pad 22: Net-(IC10-Pad22) -> DA0
- IC10 pad 33: Net-(IC10-Pad33) -> VCLK1
- IC10 pad 38: /Video/~HS -> HS
- IC39 pad 8: /DA0' -> DA0
- IC39 pad 9: /~NHS -> HS
- IC5 pad 40: /~NHS -> HS
- IC6 pad 10: /SOUND -> Net-(D5-Pad2)
- PL6 pad 6: /VIDEO -> LUMA
- PL6 pad 7: /SOUND -> SOUND
- PL6 pad 9: /MOD -> CHROMA
- R26 pad 2: /SOUND -> Net-(D5-Pad2)
- R41 pad 1: Net-(C20-Pad1) -> Net-(D5-Pad2)
- R41 pad 2: +5V -> SOUND
Routing:
- net GND: track 0.00 -> 1767.3 mm
- net +5V: track 0.00 -> 1731.2 mm, vias 0 -> 1
- net +12V: track 0.00 -> 548.4 mm, vias 0 -> 1
- net /~RESET: track 0.00 -> 523.4 mm, vias 0 -> 6
- net /PIAs/~BUSY: track 0.00 -> 475.8 mm, vias 0 -> 1
- net /D1: track 0.00 -> 459.7 mm, vias 0 -> 5
- net /D3: track 0.00 -> 453.4 mm, vias 0 -> 2
- net atx_on: track 0.00 -> 430.6 mm
- net /D2: track 0.00 -> 429.1 mm, vias 0 -> 2
- net /PIAs/STROBE: track 0.00 -> 428.0 mm, vias 0 -> 1
- net /D6: track 0.00 -> 420.5 mm, vias 0 -> 3
- net /D4: track 0.00 -> 412.8 mm, vias 0 -> 6
- net /D5: track 0.00 -> 404.3 mm, vias 0 -> 4
- net /E: track 0.00 -> 401.3 mm, vias 0 -> 2
- net /R~W~: track 0.00 -> 398.8 mm, vias 0 -> 3
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- added copper zone on B.Cu, net GND
- added copper zone on F.Cu, net GND
Other:
- board size 333.2 x 229.3 mm -> 333.2 x 165.9 mm
- board text added: "3/10/2022 - Dan Werner Dragon/CoCo V0.2"
- board text removed: "3/8/2022 - D.Werner Modified layout and ATX Power"
- board text removed: "ORIGINAL © DRAGON DATA LTD. 1983"

Commit message: Bug fixes and add Floppy Controller
Parts:
- removed D10, D19, D9: 1N914, Diode_THT:D_DO-35_SOD27_P7.62mm_Horizontal
- removed G***: LOGO, logo:we_small_neg
- removed PL8: Serial, dragon64:DIN-7_DELTRON_671-0701_Horizontal
- removed R84: 1K5, Resistor_THT:R_Axial_DIN0207_L6.3mm_D2.5mm_P7.62mm_Horizontal
- removed REG1: LM79L05_TO92, Package_TO_SOT_THT:TO-92
- removed Y1: 14.31818Mhz, Crystal:Crystal_HC49-U_Vertical
- added C48: 1u, Capacitor_THT:C_Disc_D7.5mm_W2.5mm_P5.00mm, F.Cu at (22.5, 10.4)
- added C49: 0.1uf, Capacitor_THT:C_Disc_D7.5mm_W2.5mm_P5.00mm, F.Cu at (78.9, 19.8)
- added C54: 1u, Capacitor_THT:CP_Radial_D4.0mm_P2.00mm, F.Cu at (9.30, 51.3)
- added C66: .01u, Capacitor_THT:C_Disc_D7.5mm_W2.5mm_P5.00mm, F.Cu at (305.3, 142.5)
- added C72: .01u, Capacitor_THT:C_Disc_D7.5mm_W2.5mm_P5.00mm, F.Cu at (283.2, 104.0)
- added C73: .01u, Capacitor_THT:C_Disc_D7.5mm_W2.5mm_P5.00mm, F.Cu at (241.9, 132.6)
- added C74: .01u, Capacitor_THT:C_Disc_D7.5mm_W2.5mm_P5.00mm, F.Cu at (259.7, 102.7)
- added C75: .01u, Capacitor_THT:C_Disc_D7.5mm_W2.5mm_P5.00mm, F.Cu at (317.7, 83.1)
- added C76: .01u, Capacitor_THT:C_Disc_D7.5mm_W2.5mm_P5.00mm, F.Cu at (317.9, 79.3)
- added C77: 8-70pf, Capacitor_THT:C_Radial_D6.3mm_H7.0mm_P2.50mm, F.Cu at (273.6, 143.0)
- added C78: 10nf, Capacitor_THT:C_Disc_D7.5mm_W2.5mm_P5.00mm, F.Cu at (240.9, 167.1)
- added D6: 1N4148, Diode_THT:D_DO-35_SOD27_P7.62mm_Horizontal, F.Cu at (29.6, 2.23)
- added D7: 1N4148, Diode_THT:D_DO-35_SOD27_P7.62mm_Horizontal, F.Cu at (29.6, -0.85)
- added D8: 1N914, Diode_THT:D_DO-35_SOD27_P7.62mm_Horizontal, F.Cu at (247.8, 159.4)
- added J4: DB9_Male, Connector_Dsub:DSUB-9_Male_Horizontal_P2.77x2.84mm_EdgePinOffset4.94mm_Housed_MountingHolesOffset7.48mm, F.Cu at (190.6, -22.0)
- added J5: DISK ROM ENABLE, Connector_PinHeader_2.54mm:PinHeader_1x02_P2.54mm_Vertical, F.Cu at (264.9, 59.3)
- added J6: Floppy Interface, Connector_IDC:IDC-Header_2x17_P2.54mm_Vertical, F.Cu at (187.8, 167.1)
- added R42: 100K, Resistor_THT:R_Axial_DIN0207_L6.3mm_D2.5mm_P7.62mm_Horizontal, F.Cu at (22.7, 1.13)
- added R43: 750, Resistor_THT:R_Axial_DIN0207_L6.3mm_D2.5mm_P7.62mm_Horizontal, F.Cu at (84.0, 23.6)
- added R44: 1K, Resistor_THT:R_Axial_DIN0207_L6.3mm_D2.5mm_P7.62mm_Horizontal, F.Cu at (240.2, 163.3)
- added R45: 150, Resistor_THT:R_Axial_DIN0207_L6.3mm_D2.5mm_P7.62mm_Horizontal, F.Cu at (325.9, 125.9)
- added R46: 150, Resistor_THT:R_Axial_DIN0207_L6.3mm_D2.5mm_P7.62mm_Horizontal, F.Cu at (325.9, 133.9)
- added R47: 150, Resistor_THT:R_Axial_DIN0207_L6.3mm_D2.5mm_P7.62mm_Horizontal, F.Cu at (318.2, 142.0)
- added R48: 150, Resistor_THT:R_Axial_DIN0207_L6.3mm_D2.5mm_P7.62mm_Horizontal, F.Cu at (318.2, 158.2)
- added RV1: 10K-Read, Potentiometer_THT:Potentiometer_Vishay_T73YP_Vertical, F.Cu at (213.8, 152.8)
- added RV2: 10K-Write, Potentiometer_THT:Potentiometer_Vishay_T73YP_Vertical, F.Cu at (204.2, 152.8)
- added U10: WD2797, Package_DIP:DIP-40_W15.24mm, F.Cu at (307.4, 155.4)
- added U3: 74LS00, Package_DIP:DIP-14_W7.62mm_Socket_LongPads, F.Cu at (253.3, 109.3)
- added U4: 74LS07, Package_DIP:DIP-14_W7.62mm_Socket_LongPads, F.Cu at (311.7, 88.7)
- added U5: 27C64, Package_DIP:DIP-28_W15.24mm_Socket_LongPads, F.Cu at (286.1, 57.1)
- added U6: 74LS04, Package_DIP:DIP-14_W7.62mm_Socket_LongPads, F.Cu at (277.6, 109.1)
- added U7: 74LS139, Package_DIP:DIP-16_W7.62mm_Socket_LongPads, F.Cu at (312.0, 56.0)
- added U8: 74LS06N, Package_DIP:DIP-14_W7.62mm_Socket_LongPads, F.Cu at (185.5, 138.6)
- added U9: 74LS174, Package_DIP:DIP-16_W7.62mm_Socket_LongPads, F.Cu at (312.0, 28.8)
- added X1: 14.31818Mhz, Package_DIP:DIP-14_W7.62mm_Socket_LongPads, F.Cu at (130.9, -17.9)
- added X3: 4Mhz, Package_DIP:DIP-14_W7.62mm_Socket_LongPads, F.Cu at (240.3, 138.1)
- C36: value 100uf -> 47uf
- C37: value 390pf -> 100pf
- C55: value 33uf 16V -> .01u; footprint Capacitor_THT:CP_Radial_D4.0mm_P2.00mm -> Capacitor_THT:C_Disc_D7.5mm_W2.5mm_P5.00mm
- C65: value 22p -> .01u
- C70, C71: value 1uf -> .01u; footprint Capacitor_THT:CP_Radial_D4.0mm_P2.00mm -> Capacitor_THT:C_Disc_D7.5mm_W2.5mm_P5.00mm
- C8: value .1u -> 1u
- D11: value 1N914 -> 1N4148
- Q1: footprint Package_TO_SOT_THT:TO-92_Wide -> logo:TO-92_HandSolder_FIXED
- Q2, Q3: footprint Package_TO_SOT_THT:TO-18-3 -> logo:TO-18-3_FIXED
- R10: value 4K7 -> 1K
- R9: value 4K7 -> 10K
- U2: footprint Package_DIP:DIP-14_W7.62mm_LongPads -> Package_DIP:DIP-14_W7.62mm_Socket_LongPads
- moved R10 295.7 mm to (318.2, 150.1)
- moved R9 281.0 mm to (306.7, 73.3), turned to 90 degrees
- moved J1 214.1 mm to (99.9, 165.8)
- moved C71 199.8 mm to (260.7, 142.8)
- moved C61 180.5 mm to (121.8, -1.70), turned to 180 degrees
- moved C55 167.9 mm to (318.2, 23.8)
- moved C70 111.8 mm to (191.7, 131.1), turned to 180 degrees
- moved C26 43.3 mm to (90.1, -10.5)
- moved H2 40.0 mm to (4.00, 169.0)
- moved H6 40.0 mm to (327.0, 169.0)
- moved C67 34.3 mm to (255.1, 96.0)
- moved C64 29.5 mm to (273.4, 99.5)
- moved C65 27.5 mm to (290.7, 52.1), turned to 0 degrees
- moved PL7 6.69 mm to (255.9, 10.6)
- moved J2 5.39 mm to (151.8, -25.9)
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Connections:
- net /A0 renamed A0
- net /A1 renamed A1
- net /A10 renamed A10
- net /A11 renamed A11
- net /A12 renamed A12
- net /A2 renamed A2
- net /A3 renamed A3
- net /A4 renamed A4
- net /A5 renamed A5
- net /A6 renamed A6
- net /A7 renamed A7
- net /A8 renamed A8
- net /A9 renamed A9
- net /CART renamed CART
- net /E renamed E
- net /P2 renamed P2
- net /Q renamed Q
- net /ROM2 renamed ROM2
- net /R~W~ renamed R~W~
- net /~NMI renamed ~NMI
- C25 pad 1: Net-(C25-Pad1) -> GND
- C55 pad 1: /~RESET -> +5V
- C65 pad 1: /XL3_B -> +5V
- C70 pad 1: -5V -> +5V
- C71 pad 1: -12V -> +5V
- C8 pad 2: RES_IN -> ~RESET
- D11 pad 2: /~RESET -> ~RESET
- IC10 pad 12: (no net) -> FS
- IC11 pad 4: /~RESET -> ~RESET
- IC38 pad 37: /~RESET -> ~RESET
- IC39 pad 5: /XL3_B -> GND
- IC39 pad 6: /XL3_A -> Net-(IC39-Pad6)
- IC5 pad 34: /~RESET -> ~RESET
- IC8 pad 34: /~RESET -> ~RESET
- J1 pad 12: -12V -> (no net)
- PL7 pad 5: /~RESET -> ~RESET
- PL9 pad 5: /~RESET -> ~RESET
- R10 pad 1: /Serial/S+12V -> Net-(R10-Pad1)
- R10 pad 2: +12V -> +5V
- R17 pad 1: RES_IN -> +5V
- R17 pad 2: +5V -> ~RESET
- R9 pad 1: /Serial/S-12V -> +5V
- R9 pad 2: -12V -> Net-(J5-Pad1)
- U1 pad 2: Net-(C25-Pad1) -> Net-(C54-Pad1)
- U2 pad 10: (no net) -> Net-(R43-Pad1)
Routing:
- net GND: track 1767.3 -> 0.00 mm
- net +5V: track 1731.2 -> 0.00 mm, vias 1 -> 0
- net +12V: track 548.4 -> 0.00 mm, vias 1 -> 0
- net /~RESET: track 523.4 -> 0.00 mm, vias 6 -> 0
- net /PIAs/~BUSY: track 475.8 -> 0.00 mm, vias 1 -> 0
- net /D1: track 459.7 -> 0.00 mm, vias 5 -> 0
- net /D3: track 453.4 -> 0.00 mm, vias 2 -> 0
- net atx_on: track 430.6 -> 0.00 mm
- net /D2: track 429.1 -> 0.00 mm, vias 2 -> 0
- net /PIAs/STROBE: track 428.0 -> 0.00 mm, vias 1 -> 0
- net /D6: track 420.5 -> 0.00 mm, vias 3 -> 0
- net /D4: track 412.8 -> 0.00 mm, vias 6 -> 0
- net /D5: track 404.3 -> 0.00 mm, vias 4 -> 0
- net E: track 401.3 -> 0.00 mm, vias 2 -> 0
- net R~W~: track 398.8 -> 0.00 mm, vias 3 -> 0
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- removed copper zone on B.Cu, net GND
- removed copper zone on F.Cu, net GND
Other:
- board size 333.2 x 165.9 mm -> 333.2 x 205.9 mm
- board text added: "4/09/2022 - Dan Werner Dragon/CoCo V0.5"
- board text removed: "3/10/2022 - Dan Werner Dragon/CoCo V0.2"

Commit message: add case
Parts:
- moved C72 115.8 mm to (169.7, 127.1)
- moved U6 115.8 mm to (164.1, 132.3)
- moved C65 60.5 mm to (294.4, 112.5), turned to 270 degrees
- moved U5 50.9 mm to (289.4, 107.9), turned to 270 degrees
- moved J1 45.7 mm to (145.6, 166.1)
- moved C74 38.9 mm to (228.2, 125.6)
- moved U3 38.9 mm to (221.8, 132.2)
- moved C64 28.9 mm to (245.0, 105.0)
- moved C66 26.2 mm to (313.0, 167.6)
- moved J6 10.6 mm to (177.5, 164.9)
- moved RV1 6.37 mm to (211.3, 146.9)
- moved C71 6.37 mm to (258.1, 137.0)
- moved R44 6.37 mm to (237.7, 157.5)
- moved RV2 6.37 mm to (201.6, 146.9)
- moved C73 6.37 mm to (239.4, 126.7)
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
Commit message: enclosure design work
Parts:
- moved U10 130.0 mm to (178.4, 119.5), turned to 0 degrees
- moved C74 99.6 mm to (128.6, 127.6)
- moved U6 99.6 mm to (64.5, 133.6)
- moved C73 99.6 mm to (139.8, 127.6)
- moved C78 99.6 mm to (138.7, 162.1)
- moved D8 99.6 mm to (145.7, 154.4)
- moved J6 99.6 mm to (77.9, 165.7)
- moved R44 99.6 mm to (138.1, 158.3)
- moved U8 99.6 mm to (83.3, 133.6)
- moved X3 99.6 mm to (138.2, 133.1)
- moved RV1 99.6 mm to (111.7, 147.8)
- moved RV2 99.6 mm to (102.0, 147.8)
- moved U3 99.6 mm to (122.3, 133.0)
- moved C72 99.6 mm to (70.1, 127.6)
- moved C70 99.4 mm to (89.7, 127.6)
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
Commit message: PCB layout work
Parts:
- moved R9 155.2 mm to (170.1, 146.9)
- moved U7 155.2 mm to (175.4, 129.6)
- moved C76 143.5 mm to (181.6, 124.5)
- moved C55 100.5 mm to (318.2, 124.4)
- moved U9 100.5 mm to (312.0, 129.4)
- moved C56 24.5 mm to (317.6, 23.9)
- moved IC35 24.5 mm to (311.3, 29.4)
- moved C65 22.2 mm to (259.4, 121.1)
- moved C66 22.2 mm to (285.7, 163.4)
- moved C71 22.2 mm to (210.6, 114.3)
- moved C77 22.2 mm to (233.1, 123.3)
- moved J5 22.2 mm to (263.9, 114.3)
- moved R10 22.2 mm to (284.6, 149.6)
- moved R45 22.2 mm to (292.2, 125.3)
- moved R46 22.2 mm to (292.2, 133.4)
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
Commit message: enclosure design work
Parts:
- moved J6 248.3 mm to (325.4, 145.7), turned to 180 degrees
- moved RV2 244.8 mm to (323.8, 44.0), turned to 90 degrees
- moved RV1 240.5 mm to (323.8, 34.3), turned to 90 degrees
- moved C56 161.5 mm to (194.3, 128.2)
- moved IC35 161.4 mm to (188.0, 133.6)
- moved C57 154.3 mm to (174.6, 128.2)
- moved IC25 154.2 mm to (168.3, 133.6)
- moved C38 150.0 mm to (143.7, 128.2)
- moved IC20 149.9 mm to (142.4, 133.6)
- moved U10 131.6 mm to (291.0, 23.6)
- moved C71 131.6 mm to (300.9, 18.7)
- moved C78 121.1 mm to (257.5, 110.4)
- moved D8 121.1 mm to (264.5, 102.7)
- moved C73 121.1 mm to (258.6, 75.8)
- moved R44 121.1 mm to (256.9, 106.6)
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
Commit message: pcb cleanup and readme
Parts:
- moved U8 219.2 mm to (302.5, 133.6)
- moved LK1 210.7 mm to (13.3, 136.9)
- moved IC36 204.3 mm to (26.0, 140.4)
- moved R70 182.8 mm to (63.9, 140.6), turned to 270 degrees
- moved R64 176.5 mm to (68.5, 140.5), turned to 270 degrees
- moved C38 161.9 mm to (97.6, -27.0), turned to 180 degrees
- moved U6 161.3 mm to (225.7, 133.6)
- moved PL1 150.2 mm to (42.7, -14.2)
- moved C57 146.5 mm to (32.3, 163.1)
- moved R71 144.5 mm to (310.2, 18.1)
- moved IC35 138.6 mm to (49.5, 140.4)
- moved J1 136.5 mm to (190.0, 167.6)
- moved IC25 121.8 mm to (93.2, 37.8)
- moved R80 115.2 mm to (216.9, -10.0)
- moved R81 115.2 mm to (216.9, -7.03)
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Other:
- net class GND added: clearance 0.3048, trace_width 0.762, via_dia 0.8, via_drill 0.4
- net class V12 added: clearance 0.3048, trace_width 0.5, via_dia 0.8, via_drill 0.4
- net class VCC added: clearance 0.3048, trace_width 1, via_dia 0.8, via_drill 0.4
- net class crystal removed
- net class port-power removed
- net class power+12v removed
- net class power+5v removed
- net class power-12v removed
- net class power-5v removed
- net class power-gnd removed
- net class power-mot removed
- net class video removed
- board text added: "4/18/2022 - Dan Werner Dragon/CoCo V0.5"
- board text removed: "4/09/2022 - Dan Werner Dragon/CoCo V0.5"

Commit message: pcb routing
Parts:
- moved J1 133.0 mm to (57.8, 152.7)
- moved R9 108.9 mm to (282.7, 42.9), turned to 270 degrees
- moved U3 107.1 mm to (301.6, 103.4)
- moved C62 107.0 mm to (307.9, 98.5)
- moved C67 102.2 mm to (164.8, 109.0), turned to 90 degrees
- moved C74 97.8 mm to (136.4, 67.5)
- moved C33 97.0 mm to (151.5, 67.5), turned to 180 degrees
- moved C57 82.0 mm to (88.5, 103.3)
- moved IC36 82.0 mm to (82.2, 80.7)
- moved C72 76.7 mm to (103.5, 103.0)
- moved IC35 76.7 mm to (97.2, 80.4)
- moved R64 76.7 mm to (116.2, 80.5)
- moved R70 76.7 mm to (111.6, 80.6)
- moved IC7 73.1 mm to (145.2, 73.3)
- moved C27 66.8 mm to (68.2, 138.8), turned to 0 degrees
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