File: Dragon64Board/dragon64.kicad_pcb (KiCad board)
At the start: 2 copper layers, 333.2 x 205.9 mm, 226 parts, among them IC1 74LS244, IC10 6847, IC11 6551, IC15 4164, IC16 4164, IC2 LM393, IC20 74LS273, IC21 4164, IC22 4164, IC25 74LS244, IC26 4164, IC27 4164, IC32 4164, IC33 4164, IC34 27C128, IC35 74LS00, IC36 74LS02, IC37 27C128, IC38 MC6809E, IC39 6883, IC4 4050, IC40 74LS138, IC5 6821, IC6 4529, IC7 4069, IC8 6821, J1 ATX, J2 TTL Serial Connector, J3 composite on luma, J4 DB9_Male, J5 DISK ROM ENABLE, J6 Floppy Interface, Q1 BC557, Q2 2N2222, Q3 2N2222, U1 MAX232, U10 WD2797, U2 MC1372, U3 74LS00, U4 74LS07, U5 27C64, U6 74LS04, U7 74LS139, U8 74LS06N, U9 74LS174, X1 14.31818Mhz, X3 4Mhz, Y2 1.8432Mhz

Commit message: PCB updates
Parts:
- removed X3: 4Mhz, Package_DIP:DIP-14_W7.62mm_Socket_LongPads
- added C2: 0.22uf, Capacitor_THT:C_Disc_D7.5mm_W2.5mm_P5.00mm, F.Cu at (310.2, 53.3)
- added C5: 47pf, Capacitor_THT:C_Disc_D7.5mm_W2.5mm_P5.00mm, F.Cu at (294.5, 80.5)
- added C68: 10nf, Capacitor_THT:C_Disc_D7.5mm_W2.5mm_P5.00mm, F.Cu at (310.6, 69.7)
- added R49: 1K, Resistor_THT:R_Axial_DIN0207_L6.3mm_D2.5mm_P7.62mm_Horizontal, F.Cu at (305.2, 74.2)
- added R50: 1K, Resistor_THT:R_Axial_DIN0207_L6.3mm_D2.5mm_P7.62mm_Horizontal, F.Cu at (319.4, 74.4)
- added U11: 74LS74, Package_DIP:DIP-14_W7.62mm_Socket_LongPads, F.Cu at (317.4, 45.4)
- added Y1: 4mhz, Crystal:Crystal_HC49-U_Vertical, F.Cu at (306.0, 80.6)
- C77: footprint Capacitor_THT:C_Radial_D6.3mm_H7.0mm_P2.50mm -> dragon64:c_trimmer-10
- moved C73 7.73 mm to (323.7, 65.2), turned to 180 degrees
- moved C77 5.41 mm to (256.0, -5.30)
Connections:
- net Net-(J1-Pad1) renamed +3V3
- D8 pad 1: Net-(D8-Pad1) -> Net-(C2-Pad1)
- R44 pad 2: Net-(D8-Pad1) -> Net-(C2-Pad1)
- U10 pad 23: Net-(D8-Pad1) -> Net-(C2-Pad2)
- U10 pad 24: Net-(U10-Pad24) -> DSKCLK
- U6 pad 10: (no net) -> Net-(R50-Pad1)
- U6 pad 11: (no net) -> Net-(C68-Pad1)
- U6 pad 8: DISKMOTOR -> Net-(C68-Pad2)
- U6 pad 9: Net-(U6-Pad9) -> Net-(C5-Pad2)
- U8 pad 12: (no net) -> DISKMOTOR
- U8 pad 13: (no net) -> Net-(U8-Pad13)
- U9 pad 7: Net-(U6-Pad9) -> Net-(U8-Pad13)
Routing:
- net GND: track 0.00 -> 2495.9 mm, vias 0 -> 2
- net +5V: track 0.00 -> 2291.2 mm, vias 0 -> 2
- net D4: track 0.00 -> 568.7 mm, vias 0 -> 5
- net D5: track 0.00 -> 536.8 mm, vias 0 -> 6
- net D0: track 0.00 -> 536.1 mm, vias 0 -> 2
- net D7: track 0.00 -> 534.0 mm, vias 0 -> 3
- net D3: track 0.00 -> 523.0 mm, vias 0 -> 5
- net A0: track 0.00 -> 505.7 mm, vias 0 -> 2
- net D2: track 0.00 -> 498.2 mm, vias 0 -> 5
- net D6: track 0.00 -> 497.7 mm, vias 0 -> 4
- net A1: track 0.00 -> 496.7 mm, vias 0 -> 1
- net D1: track 0.00 -> 489.3 mm, vias 0 -> 2
- net ~RESET: track 0.00 -> 483.1 mm, vias 0 -> 2
- net R~W~: track 0.00 -> 471.2 mm, vias 0 -> 3
- net E: track 0.00 -> 465.2 mm, vias 0 -> 3
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- added copper zone on B.Cu, net GND
- added copper zone on F.Cu, net GND
Other:
- board text added: "6/18/2022 - Dan Werner Dragon/CoCo V0.7"
- board text removed: "5/30/2022 - Dan Werner Dragon/CoCo V0.6"

Commit message: version 1.0 cleanup
Parts:
- C77: value 8-70pf -> 8-70pf - Floppy Adjust
- J1: value ATX -> Screw_Terminal_01x03; footprint Connector_Molex:Molex_Mini-Fit_Jr_5566-20A_2x10_P4.20mm_Vertical -> TerminalBlock_RND:TerminalBlock_RND_205-00277_1x03_P5.00mm_Vertical
- LK1: value ~ -> RAM SIZE SELECT
- PL6: value Power/Video -> Video/Audio
- moved J1 25.0 mm to (27.9, 143.1), turned to 0 degrees
Connections:
- J1 pad 1: +3V3 -> +12V
- J1 pad 2: +3V3 -> GND
- J1 pad 3: GND -> +5V
- PL6 pad 1: atx_on -> GND
Routing:
- net atx_on: track 204.1 -> 0.00 mm
- net +5V: track 2291.2 -> 2259.8 mm
- net +3V3: track 9.70 -> 0.00 mm
- net GND: track 2495.9 -> 2487.9 mm
- net +12V: track 451.0 -> 453.8 mm
Other:
- board text added: "+12V"
- board text added: "+5V"
- board text added: "7/1/2022 - Dan Werner Dragon/CoCo V1.0"
- board text added: "GND"
- board text added: "POWER"
- board text removed: "6/18/2022 - Dan Werner Dragon/CoCo V0.7"
