File: Dragon64Board/dragon64.kicad_pcb (KiCad board)
At the start: 2 copper layers, 333.2 x 205.9 mm, 232 parts, among them IC1 74LS244, IC10 6847, IC11 6551, IC15 4164, IC16 4164, IC2 LM393, IC20 74LS273, IC21 4164, IC22 4164, IC25 74LS244, IC26 4164, IC27 4164, IC32 4164, IC33 4164, IC34 27C128, IC35 74LS00, IC36 74LS02, IC37 27C128, IC38 MC6809E, IC39 6883, IC4 4050, IC40 74LS138, IC5 6821, IC6 4529, IC7 4069, IC8 6821, J1 Screw_Terminal_01x03, J2 TTL Serial Connector, J3 composite on luma, J4 DB9_Male, J5 DISK ROM ENABLE, J6 Floppy Interface, Q1 BC557, Q2 2N2222, Q3 2N2222, U1 MAX232, U10 WD2797, U11 74LS74, U2 MC1372, U3 74LS00, U4 74LS07, U5 27C64, U6 74LS04, U7 74LS139, U8 74LS06N, U9 74LS174, X1 14.31818Mhz, Y1 4mhz, Y2 1.8432Mhz

Commit message: version 1.0 cleanup
Other:
- board text added: "https://github.com/danwerner21/Dragon64"
Changed lines of the file:
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@@
   (general
     (thickness 1.6)
-    (drawings 27)
+    (drawings 28)
     (tracks 6665)
     (zones 0)
@@
   (page A3)
   (layers
-    (0 F.Cu signal)
-    (31 B.Cu signal)
+    (0 F.Cu signal hide)
+    (31 B.Cu signal hide)
     (32 B.Adhes user)
     (33 F.Adhes user)
@@
   )
   (setup
-    (last_trace_width 1.016)
+    (last_trace_width 0.2032)
     (user_trace_width 0.254)
     (user_trace_width 0.381)
@@
     )
   )
+  (gr_text https://github.com/danwerner21/Dragon64 (at 251.6 164.8) (layer F.SilkS)
+    (effects (font (size 1.5 1.5) (thickness 0.3)))
+  )
   (gr_text +5V (at 38.2 155.5 90) (layer F.SilkS)
     (effects (font (size 1.5 1.5) (thickness 0.3)))
@@
   (via (at 280.3333 56.2928) (size 0.8) (layers F.Cu B.Cu) (net 61))
   (via (at 118.3011 74.9347) (size 0.8) (layers F.Cu B.Cu) (net 61))
+  (segment (start 31.7748 -23.3748) (end 31.7748 -24.9248) (width 1.016) (layer F.Cu) (net 61))
+  (segment (start 31.7748 -23.3748) (end 38.2954 -23.3748) (width 0.762) (layer F.Cu) (net 61))
+  (segment (start 31.7748 -24.9248) (end 31.775 -24.925) (width 1.016) (layer F.Cu) (net 61))
+  (segment (start 25.7052 -23.3748) (end 31.7748 -23.3748) (width 0.762) (layer F.Cu) (net 61))
+  (segment (start 32.9 143.1) (end 32.9 152.2) (width 1.016) (layer F.Cu) (net 61))
+  (segment (start 32.9 152.2) (end 46.4 165.7) (width 1.016) (layer F.Cu) (net 61))
+  (segment (start 40.8361 160.0181) (end 46.4 165.7) (width 0.762) (layer F.Cu) (net 61))
+  (segment (start 46.4 165.7) (end 50.718 169.9) (width 0.762) (layer F.Cu) (net 61))
   (segment (start 91.4622 76.8076) (end 91.8004 77.1458) (width 0.2032) (layer F.Cu) (net 62))
   (segment (start 91.8004 77.1458) (end 125.9159 77.1458) (width 0.2032) (layer F.Cu) (net 62))
@@
   (via (at 151.3497 27.71) (size 0.8) (layers F.Cu B.Cu) (net 157))
   (via (at 57.0363 -2.1739) (size 0.8) (layers F.Cu B.Cu) (net 157))
-  (segment (start 31.7748 -23.3748) (end 31.7748 -24.9248) (width 1.016) (layer F.Cu) (net 61))
-  (segment (start 31.7748 -23.3748) (end 38.2954 -23.3748) (width 0.762) (layer F.Cu) (net 61))
-  (segment (start 31.7748 -24.9248) (end 31.775 -24.925) (width 1.016) (layer F.Cu) (net 61))
-  (segment (start 25.7052 -23.3748) (end 31.7748 -23.3748) (width 0.762) (layer F.Cu) (net 61))
-  (segment (start 32.9 143.1) (end 32.9 152.2) (width 1.016) (layer F.Cu) (net 61))
-  (segment (start 32.9 152.2) (end 46.4 165.7) (width 1.016) (layer F.Cu) (net 61))
-  (segment (start 40.8361 160.0181) (end 46.4 165.7) (width 0.762) (layer F.Cu) (net 61))
-  (segment (start 46.4 165.7) (end 50.718 169.9) (width 0.762) (layer F.Cu) (net 61))
   (segment (start 5.75 -11.855) (end 5.75 -12.9601) (width 0.2032) (layer B.Cu) (net 158))
   (segment (start 29.235 -24.925) (end 28.0799 -24.925) (width 0.2032) (layer B.Cu) (net 158))

Commit message: version 1.0 cleanup
Other:
- board text added: "7/1/2022 - Dan Werner Dragon 64 V1.0"
- board text removed: "7/1/2022 - Dan Werner Dragon/CoCo V1.0"
Changed lines of the file:
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@@
   (gr_arc (start 0.25 175.746) (end -0.004 175.746) (angle -90) (layer Edge.Cuts) (width 0.05))
   (gr_arc (start 332.95 175.8) (end 332.95 176) (angle -90) (layer Edge.Cuts) (width 0.05))
-  (gr_text "7/1/2022 - Dan Werner Dragon/CoCo V1.0\n" (at 265.05 168.69) (layer F.SilkS)
+  (gr_text "7/1/2022 - Dan Werner Dragon 64 V1.0\n" (at 265.05 168.69) (layer F.SilkS)
     (effects (font (size 2.25 2.25) (thickness 0.25)))
   )
