File: Dragon64Board/pia.sch (KiCad schematic (older format))
At the start: 74 parts, among them IC1 74LS244, IC2 LM393, IC36 74LS02, IC4 4050, IC5 6821, IC6 4529, IC7 4069, IC8 6821

Commit message: PAL to NTSC
Parts:
- added D5: 1N4148, Diode_THT:D_DO-35_SOD27_P7.62mm_Horizontal, symbol Device:D
- added R41: 1K, Resistor_THT:R_Axial_DIN0207_L6.3mm_D2.5mm_P7.62mm_Horizontal, symbol Device:R
Connections:
- net SOUND: now also D5.1 (K), R41.2; no longer IC6.10 (W), R26.2
- net ~FS renamed FS
- net ~NHS renamed HS
- new net: D5.2 (A), IC6.10 (W), R26.2, R41.1
Changed lines of the file:
@@
 Text HLabel 1150 10850 0    50   Input ~ 0
 CART
-Text HLabel 3350 2600 2    50   Input ~ 0
-~NHS
 Wire Wire Line
 	4000 1200 4000 1700
@@
 	7800 9350 7400 9350
 Connection ~ 7400 9350
-Text HLabel 3350 3900 2    50   Input ~ 0
-~FS
 Wire Wire Line
 	3350 3900 3250 3900
@@
 Wire Wire Line
 	4400 2000 5550 2000
-Text HLabel 15050 6000 2    50   Output ~ 0
-SOUND
 Wire Wire Line
 	12900 5850 12900 6000
@@
 Connection ~ 14700 6000
 Wire Wire Line
-	14700 6000 15050 6000
-Wire Wire Line
 	1900 6750 1900 7000
 Wire Wire Line
@@
 NoConn ~ 13800 8650
 NoConn ~ -2900 2550
+Text GLabel 3350 2600 2    50   Input ~ 0
+HS
+$Comp
+L Device:R R?
+U 1 1 62C31866
+P 15350 6000
+AR Path="/62C31866" Ref="R?"  Part="1"
+AR Path="/60168BB0/62C31866" Ref="R41"  Part="1"
+F 0 "R41" V 15450 5950 50  0000 L CNN
+F 1 "1K" V 15250 5950 50  0000 L CNN
+F 2 "Resistor_THT:R_Axial_DIN0207_L6.3mm_D2.5mm_P7.62mm_Horizontal" V 15280 6000 50  0001 C CNN
+F 3 "~" H 15350 6000 50  0001 C CNN
+	1    15350 6000
+	0    -1   -1   0
+$EndComp
+Wire Wire Line
+	14700 6000 15200 6000
+Wire Wire Line
+	15500 6000 15650 6000
+$Comp
+L Device:D D5
+U 1 1 62C9324A
+P 15350 5750
+F 0 "D5" H 15350 5533 50  0000 C CNN
+F 1 "1N4148" H 15350 5624 50  0000 C CNN
+F 2 "Diode_THT:D_DO-35_SOD27_P7.62mm_Horizontal" H 15350 5750 50  0001 C CNN
+F 3 "~" H 15350 5750 50  0001 C CNN
+	1    15350 5750
+	-1   0    0    1
+$EndComp
+Wire Wire Line
+	15200 5750 15200 6000
+Connection ~ 15200 6000
+Wire Wire Line
+	15500 5750 15500 6000
+Connection ~ 15500 6000
+Text GLabel 3350 3900 2    50   Input ~ 0
+FS
+Text GLabel 15650 6000 2    50   Input ~ 0
+SOUND
 $EndSCHEMATC

Commit message: Bug fixes and add Floppy Controller
Other:
- note removed: "**"
- note removed: "** L3, L4, C68, C69 OPTIONAL\nFOR SECOND JOYSTICK BUTTON"
Changed lines of the file:
@@
 $Descr A3 16535 11693
 encoding utf-8
-Sheet 4 5
-Title "Dragon CPU 64K (PAL)"
-Date "2020-12-21"
+Sheet 4 6
+Title "Dragon CPU 64K"
+Date "2022-04-09"
 Rev "4"
-Comp "Dragon Data Ltd."
-Comment1 "Transcribed by Ciaran Anscomb, 2020"
-Comment2 "PIAs, I/O, analogue routing"
+Comp "Originally by Dragon Data Ltd."
+Comment1 ""
+Comment2 ""
 Comment3 ""
 Comment4 ""
@@
 Text Label 11250 6150 2    50   ~ 0
 STY
-Text Notes 12000 950  0    50   ~ 0
-** L3, L4, C68, C69 OPTIONAL\nFOR SECOND JOYSTICK BUTTON
 Text Notes 9900 10550 2    39   ~ 0
 16V ELECTRO
@@
 Wire Wire Line
 	13850 1350 13850 2200
-Text Notes 12250 1250 0    50   ~ 0
-**
-Text Notes 12250 1350 0    50   ~ 0
-**
-Text Notes 11600 1650 0    50   ~ 0
-**
-Text Notes 12050 1650 0    50   ~ 0
-**
 Wire Wire Line
 	12000 2050 12000 1850

Commit message: enclosure design work
Parts:
- C2, C5, C68, C69: value .01u -> .1u
Changed lines of the file:
@@
 P 11100 1500
 F 0 "C2" H 11000 1400 50  0000 C CNN
-F 1 ".01u" H 10950 1600 50  0000 C CNN
+F 1 ".1u" H 10950 1600 50  0000 C CNN
 F 2 "Capacitor_THT:C_Disc_D7.5mm_W2.5mm_P5.00mm" H 11138 1350 50  0001 C CNN
 F 3 "~" H 11100 1500 50  0001 C CNN
@@
 P 10700 1500
 F 0 "C5" H 10600 1400 50  0000 C CNN
-F 1 ".01u" H 10550 1600 50  0000 C CNN
+F 1 ".1u" H 10550 1600 50  0000 C CNN
 F 2 "Capacitor_THT:C_Disc_D7.5mm_W2.5mm_P5.00mm" H 10738 1350 50  0001 C CNN
 F 3 "~" H 10700 1500 50  0001 C CNN
@@
 P 12150 1700
 F 0 "C68" H 12250 1800 50  0000 C CNN
-F 1 ".01u" H 12250 1600 50  0000 C CNN
+F 1 ".1u" H 12250 1600 50  0000 C CNN
 F 2 "Capacitor_THT:C_Disc_D7.5mm_W2.5mm_P5.00mm" H 12188 1550 50  0001 C CNN
 F 3 "~" H 12150 1700 50  0001 C CNN
@@
 P 11700 1700
 F 0 "C69" H 11600 1600 50  0000 C CNN
-F 1 ".01u" H 11550 1800 50  0000 C CNN
+F 1 ".1u" H 11550 1800 50  0000 C CNN
 F 2 "Capacitor_THT:C_Disc_D7.5mm_W2.5mm_P5.00mm" H 11738 1550 50  0001 C CNN
 F 3 "~" H 11700 1700 50  0001 C CNN

Commit message: add rom images
Parts:
- removed C2, C5, C68, C69: .1u, Capacitor_THT:C_Disc_D7.5mm_W2.5mm_P5.00mm, symbol Device:C
Changed lines of the file:
@@
 $EndComp
-Wire Wire Line
-	11250 1050 10700 1050
-Wire Wire Line
-	11250 1150 11100 1150
 Wire Wire Line
 	11550 1150 13450 1150
@@
 Connection ~ 14300 2900
 $Comp
-L Device:C C2
-U 1 1 60EFD0C3
-P 11100 1500
-F 0 "C2" H 11000 1400 50  0000 C CNN
-F 1 ".1u" H 10950 1600 50  0000 C CNN
-F 2 "Capacitor_THT:C_Disc_D7.5mm_W2.5mm_P5.00mm" H 11138 1350 50  0001 C CNN
-F 3 "~" H 11100 1500 50  0001 C CNN
-	1    11100 1500
-	-1   0    0    1
-$EndComp
-$Comp
-L Device:C C5
-U 1 1 60EFF2BF
-P 10700 1500
-F 0 "C5" H 10600 1400 50  0000 C CNN
-F 1 ".1u" H 10550 1600 50  0000 C CNN
-F 2 "Capacitor_THT:C_Disc_D7.5mm_W2.5mm_P5.00mm" H 10738 1350 50  0001 C CNN
-F 3 "~" H 10700 1500 50  0001 C CNN
-	1    10700 1500
-	-1   0    0    1
-$EndComp
-Wire Wire Line
-	10700 1350 10700 1050
-Connection ~ 10700 1050
-Wire Wire Line
-	10700 1050 10350 1050
-Wire Wire Line
-	11100 1350 11100 1150
-Connection ~ 11100 1150
-Wire Wire Line
-	11100 1150 10350 1150
-$Comp
-L power:GND #PWR0273
-U 1 1 60FDD8E3
-P 10900 1850
-F 0 "#PWR0273" H 10900 1600 50  0001 C CNN
-F 1 "GND" H 10905 1677 50  0000 C CNN
-F 2 "" H 10900 1850 50  0001 C CNN
-F 3 "" H 10900 1850 50  0001 C CNN
-	1    10900 1850
-	1    0    0    -1
-$EndComp
-Wire Wire Line
-	10700 1650 10900 1650
-Wire Wire Line
-	10900 1850 10900 1650
-Connection ~ 10900 1650
-Wire Wire Line
-	10900 1650 11100 1650
-$Comp
 L Connector:DIN-6 PL5
 U 1 1 5FCB0335
@@
 	0    -1   -1   0
 $EndComp
-$Comp
-L Device:C C68
-U 1 1 5FD4FBB0
-P 12150 1700
-F 0 "C68" H 12250 1800 50  0000 C CNN
-F 1 ".1u" H 12250 1600 50  0000 C CNN
-F 2 "Capacitor_THT:C_Disc_D7.5mm_W2.5mm_P5.00mm" H 12188 1550 50  0001 C CNN
-F 3 "~" H 12150 1700 50  0001 C CNN
-	1    12150 1700
-	1    0    0    -1
-$EndComp
-$Comp
-L Device:C C69
-U 1 1 5FD4FBB6
-P 11700 1700
-F 0 "C69" H 11600 1600 50  0000 C CNN
-F 1 ".1u" H 11550 1800 50  0000 C CNN
-F 2 "Capacitor_THT:C_Disc_D7.5mm_W2.5mm_P5.00mm" H 11738 1550 50  0001 C CNN
-F 3 "~" H 11700 1700 50  0001 C CNN
-	1    11700 1700
-	-1   0    0    1
-$EndComp
-Wire Wire Line
-	11700 1550 11700 1250
-Wire Wire Line
-	12150 1550 12150 1350
-Wire Wire Line
-	11700 1850 12000 1850
-Connection ~ 12000 1850
-Wire Wire Line
-	12000 1850 12150 1850
 Wire Wire Line
 	13000 1250 13000 2800
@@
 	13850 1350 13850 2200
 Wire Wire Line
-	12000 2050 12000 1850
-$Comp
-L power:GND #PWR01
-U 1 1 5FD4FBBE
-P 12000 2050
-F 0 "#PWR01" H 12000 1800 50  0001 C CNN
-F 1 "GND" H 12005 1877 50  0000 C CNN
-F 2 "" H 12000 2050 50  0001 C CNN
-F 3 "" H 12000 2050 50  0001 C CNN
-	1    12000 2050
-	1    0    0    -1
-$EndComp
-Wire Wire Line
 	13000 1250 12700 1250
 Wire Wire Line
 	13850 1350 12700 1350
-Wire Wire Line
-	12400 1350 12150 1350
-Connection ~ 12150 1350
-Wire Wire Line
-	12400 1250 11700 1250
-Connection ~ 11700 1250
 Text Label 13850 2100 0    50   ~ 0
 JL_F2
@@
 Text Label 13850 3100 0    50   ~ 0
 JR_F2
-Wire Wire Line
-	10350 1250 11700 1250
 $Comp
 L dragon64:4529 IC6
@@
 Wire Wire Line
 	11650 4850 11650 4800
-Wire Wire Line
-	10350 1350 12150 1350
 $Comp
 L Device:C_Polarized_US C19
@@
 Text GLabel 15650 6000 2    50   Input ~ 0
 SOUND
+Wire Wire Line
+	10350 1150 11250 1150
+Wire Wire Line
+	10350 1050 11250 1050
+Wire Wire Line
+	10350 1350 12400 1350
+Wire Wire Line
+	10350 1250 12400 1250
 $EndSCHEMATC
