File: Dragon64Board/_autosave-disk.sch (KiCad schematic (older format))
At the start: 25 parts, among them J5 DISK ROM ENABLE, J6 Floppy Interface, U10 WD2797, U3 74LS00, U4 74LS07, U5 27C64, U6 74LS04, U7 74LS139, U8 74LS06N, U9 74LS174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

Commit message: documentation update
Parts:
- removed C5: 10nf, Capacitor_THT:C_Disc_D7.5mm_W2.5mm_P5.00mm, symbol Device:C
- X2: value CXO_DIP14 -> 1 Mhz; footprint Oscillator:Oscillator_DIP-14 -> Package_DIP:DIP-14_W7.62mm_Socket_LongPads
Changed lines of the file:
@@
 Text GLabel 7850 2450 0    50   Input ~ 0
 D7
-$Comp
-L Device:C C?
-U 1 1 630456A4
-P 9300 4250
-AR Path="/62D1E9EB/62A00355" Ref="C?"  Part="1"
-AR Path="/62D1E9EB/630456A4" Ref="C5"  Part="1"
-F 0 "C5" V 9200 4150 50  0000 C CNN
-F 1 "10nf" V 9200 4400 50  0000 C CNN
-F 2 "Capacitor_THT:C_Disc_D7.5mm_W2.5mm_P5.00mm" H 9338 4100 50  0001 C CNN
-F 3 "~" H 9300 4250 50  0001 C CNN
-	1    9300 4250
-	0    1    1    0
-$EndComp
 NoConn ~ 5650 1650
 Wire Wire Line
@@
 U 1 1 631746F6
 P 7650 2950
-F 0 "R10" V 7600 2700 50  0000 L CNN
+F 0 "R10" V 7600 2650 50  0000 L CNN
 F 1 "1K" V 7700 2700 50  0000 L CNN
 F 2 "Resistor_THT:R_Axial_DIN0207_L6.3mm_D2.5mm_P7.62mm_Horizontal" V 7580 2950 50  0001 C CNN
@@
 P 7750 2850
 F 0 "#PWR0186" H 7750 2600 50  0001 C CNN
-F 1 "GND" V 7755 2722 50  0000 R CNN
+F 1 "GND" V 7700 2750 50  0000 R CNN
 F 2 "" H 7750 2850 50  0001 C CNN
 F 3 "" H 7750 2850 50  0001 C CNN
@@
 P 5950 1650
 F 0 "X2" H 6294 1696 50  0000 L CNN
-F 1 "CXO_DIP14" H 6294 1605 50  0000 L CNN
-F 2 "Oscillator:Oscillator_DIP-14" H 6400 1300 50  0001 C CNN
+F 1 "1 Mhz" H 6294 1605 50  0000 L CNN
+F 2 "Package_DIP:DIP-14_W7.62mm_Socket_LongPads" H 6400 1300 50  0001 C CNN
 F 3 "http://cdn-reichelt.de/documents/datenblatt/B400/OSZI.pdf" H 5850 1650 50  0001 C CNN
 	1    5950 1650
