File: Dragon64Board/disk.sch (KiCad schematic (older format))
At the start: 23 parts, among them J5 DISK ROM ENABLE, J6 Floppy Interface, U10 WD2797, U3 74LS00, U4 74LS07, U5 27C64, U6 74LS04, U7 74LS139, U8 74LS06N, U9 74LS174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

Commit message: add case
Other:
- note added: "DISK CONTROLLER IS OPTIONAL\nIF NOT NEEDED, DO NOT POPULATE THIS SHEET"
Changed lines of the file:
@@
 $EndComp
 NoConn ~ 4350 6900
+Text Notes 1800 6250 0    157  ~ 0
+DISK CONTROLLER IS OPTIONAL\nIF NOT NEEDED, DO NOT POPULATE THIS SHEET
 $EndSCHEMATC

Commit message: documentation update
Parts:
- added C2: 0.22uf, Capacitor_THT:C_Disc_D7.5mm_W2.5mm_P5.00mm, symbol Device:C
- added X2: CXO_DIP14, Package_DIP:DIP-14_W7.62mm_Socket_LongPads, symbol Oscillator:CXO_DIP14
- C5: renamed from X3; value 4Mhz -> 10nf; footprint Package_DIP:DIP-14_W7.62mm_Socket_LongPads -> Capacitor_THT:C_Disc_D7.5mm_W2.5mm_P5.00mm; symbol Oscillator:XO91 -> Device:C
Connections:
- net +5V: now also X2.14 (Vcc); no longer C5.4 (V+)
- net GND: now also X2.7 (GND); no longer C5.2 (GND)
- net at D8.1 (K), R44.2: now also C2.1; no longer U10.23 (PUMP)
- net at U10.24 (CLK): now also X2.8 (OUT); no longer C5.3 (OUT)
- new net: C2.2, U10.23 (PUMP)
Changed lines of the file:
@@
 D7
 $Comp
-L Oscillator:XO91 X3
+L Device:C C?
 U 1 1 630456A4
-P 5950 1650
-F 0 "X3" H 6294 1696 50  0000 L CNN
-F 1 "4Mhz" H 6294 1605 50  0000 L CNN
-F 2 "Package_DIP:DIP-14_W7.62mm_Socket_LongPads" H 6650 1300 50  0001 C CNN
-F 3 "http://cdn-reichelt.de/documents/datenblatt/B400/XO91.pdf" H 5850 1650 50  0001 C CNN
-	1    5950 1650
-	1    0    0    -1
+P 9300 4250
+AR Path="/62D1E9EB/62A00355" Ref="C?"  Part="1"
+AR Path="/62D1E9EB/630456A4" Ref="C5"  Part="1"
+F 0 "C5" V 9200 4150 50  0000 C CNN
+F 1 "10nf" V 9200 4400 50  0000 C CNN
+F 2 "Capacitor_THT:C_Disc_D7.5mm_W2.5mm_P5.00mm" H 9338 4100 50  0001 C CNN
+F 3 "~" H 9300 4250 50  0001 C CNN
+	1    9300 4250
+	0    1    1    0
 $EndComp
 NoConn ~ 5650 1650
@@
 	0    1    1    0
 $EndComp
-Wire Wire Line
-	10000 3950 9000 3950
 $Comp
 L Diode:1N914 D8
@@
 Wire Wire Line
 	10000 3950 10000 4150
-Connection ~ 10000 3950
 Wire Wire Line
 	10300 4150 10300 3950
@@
 Text Notes 1800 6250 0    157  ~ 0
 DISK CONTROLLER IS OPTIONAL\nIF NOT NEEDED, DO NOT POPULATE THIS SHEET
+$Comp
+L Device:C C2
+U 1 1 62A00355
+P 9350 3950
+F 0 "C2" V 9250 3850 50  0000 C CNN
+F 1 "0.22uf" V 9250 4100 50  0000 C CNN
+F 2 "Capacitor_THT:C_Disc_D7.5mm_W2.5mm_P5.00mm" H 9388 3800 50  0001 C CNN
+F 3 "~" H 9350 3950 50  0001 C CNN
+	1    9350 3950
+	0    1    1    0
+$EndComp
+Wire Wire Line
+	9000 3950 9200 3950
+Wire Wire Line
+	9500 3950 10000 3950
+Connection ~ 10000 3950
+$Comp
+L Oscillator:CXO_DIP14 X2
+U 1 1 62C24C2D
+P 5950 1650
+F 0 "X2" H 6294 1696 50  0000 L CNN
+F 1 "CXO_DIP14" H 6294 1605 50  0000 L CNN
+F 2 "Package_DIP:DIP-14_W7.62mm_Socket_LongPads" H 6400 1300 50  0001 C CNN
+F 3 "http://cdn-reichelt.de/documents/datenblatt/B400/OSZI.pdf" H 5850 1650 50  0001 C CNN
+	1    5950 1650
+	1    0    0    -1
+$EndComp
 $EndSCHEMATC

Commit message: PCB updates
Parts:
- removed X2: CXO_DIP14, Package_DIP:DIP-14_W7.62mm_Socket_LongPads, symbol Oscillator:CXO_DIP14
- added C68: 10nf, Capacitor_THT:C_Disc_D7.5mm_W2.5mm_P5.00mm, symbol Device:C
- added R49, R50: 1K, Resistor_THT:R_Axial_DIN0207_L6.3mm_D2.5mm_P7.62mm_Horizontal, symbol Device:R
- added U11: 74LS74, Package_DIP:DIP-14_W7.62mm_Socket_LongPads, symbol 74xx:74LS74
- added unit 5 of U6
- added unit 6 of U6
- added Y1: 4mhz, Crystal:Crystal_HC49-U_Vertical, symbol Device:Crystal
- C5: value 10nf -> 47pf
- C77: footprint Capacitor_THT:C_Radial_D6.3mm_H7.0mm_P2.50mm -> dragon64:c_trimmer-10
Connections:
- net +5V: now also U11.1 (~R), U11.10 (~S), U11.13 (~R), U11.14 (VCC), U11.4 (~S)
- net DISKMOTOR: now also U8.12; no longer U6.8
- net GND: now also C5.1, U11.7 (GND)
- net DSKCLK: now reaches U10.24 (CLK)
- net DSKCLK: now also U11.2 (D), U11.6 (~Q)
- net at U9.7 (Q2): now also U8.13; no longer U6.9
- net at C5.2: now also U6.9, R49.2, Y1.1
- new net: R50.1, U11.11 (C), U6.10, Y1.2
- new net: C68.1, R50.2, U6.11
- new net: C68.2, R49.1, U6.8
- new net: U11.12 (D), U11.3 (C), U11.8 (~Q)
- no-connect marks 12 -> 13
Other:
- moved on the sheet: U3E, U4F, U4G, U6D, U6G, U8F, U8G
