File: Dragon64Board/dragon64.sch (KiCad schematic (older format))
At the start: 55 parts, among them IC34 27C128, IC35 74LS00, IC36 74LS02, IC37 27C128, IC38 MC6809E, IC39 6883, IC40 74LS138, J1 ATX, X1 14.31818Mhz

Commit message: version 1.0 cleanup
Parts:
- removed J1: ATX, Connector_Molex:Molex_Mini-Fit_Jr_5566-20A_2x10_P4.20mm_Vertical, symbol Connector:ATX-20
- added J1: Screw_Terminal_01x03, TerminalBlock_RND:TerminalBlock_RND_205-00277_1x03_P5.00mm_Vertical, symbol Connector:Screw_Terminal_01x03
Connections:
- net atx_on is gone; now on net GND: PL6.1 (Pin_1)
- net +12V: now also J1.1 (Pin_1)
- net +5V: now also J1.3 (Pin_3)
- net GND: now also J1.2 (Pin_2)
- no-connect marks 11 -> 7
Changed lines of the file:
@@
 L power:+12V #PWR0253
 U 1 1 60A51415
-P 10550 1100
-F 0 "#PWR0253" H 10550 950 50  0001 C CNN
-F 1 "+12V" H 10565 1273 50  0000 C CNN
-F 2 "" H 10550 1100 50  0001 C CNN
-F 3 "" H 10550 1100 50  0001 C CNN
-	1    10550 1100
-	0    1    1    0
+P 11350 700
+F 0 "#PWR0253" H 11350 550 50  0001 C CNN
+F 1 "+12V" H 11365 873 50  0000 C CNN
+F 2 "" H 11350 700 50  0001 C CNN
+F 3 "" H 11350 700 50  0001 C CNN
+	1    11350 700
+	0    -1   -1   0
 $EndComp
 $Comp
 L power:+5V #PWR0254
 U 1 1 60A51DFB
-P 10550 1300
-F 0 "#PWR0254" H 10550 1150 50  0001 C CNN
-F 1 "+5V" H 10565 1473 50  0000 C CNN
-F 2 "" H 10550 1300 50  0001 C CNN
-F 3 "" H 10550 1300 50  0001 C CNN
-	1    10550 1300
-	0    1    1    0
+P 11350 900
+F 0 "#PWR0254" H 11350 750 50  0001 C CNN
+F 1 "+5V" H 11365 1073 50  0000 C CNN
+F 2 "" H 11350 900 50  0001 C CNN
+F 3 "" H 11350 900 50  0001 C CNN
+	1    11350 900
+	0    -1   -1   0
 $EndComp
 $Comp
 L power:GND #PWR0256
 U 1 1 60A8D968
-P 9850 2000
-F 0 "#PWR0256" H 9850 1750 50  0001 C CNN
-F 1 "GND" H 9855 1827 50  0000 C CNN
-F 2 "" H 9850 2000 50  0001 C CNN
-F 3 "" H 9850 2000 50  0001 C CNN
-	1    9850 2000
-	1    0    0    -1
+P 11050 800
+F 0 "#PWR0256" H 11050 550 50  0001 C CNN
+F 1 "GND" H 11055 627 50  0000 C CNN
+F 2 "" H 11050 800 50  0001 C CNN
+F 3 "" H 11050 800 50  0001 C CNN
+	1    11050 800
+	0    1    1    0
 $EndComp
 Wire Wire Line
@@
 $EndComp
 Wire Wire Line
-	9350 900  9150 900
-Text GLabel 9150 900  0    50   Input ~ 0
-atx_on
-Wire Wire Line
-	12150 1650 12150 1800
-Wire Wire Line
-	12150 1800 12350 1800
-Text GLabel 12350 1800 2    50   Input ~ 0
-atx_on
-Wire Wire Line
 	12050 1650 12050 2050
 Wire Wire Line
@@
 Wire Wire Line
 	12600 2050 12650 2050
-NoConn ~ 10350 900
-NoConn ~ 10350 1600
-$Comp
-L Connector:ATX-20 J1
-U 1 1 602A61BC
-P 9850 1300
-F 0 "J1" H 9850 1967 50  0000 C CNN
-F 1 "ATX" H 9850 1876 50  0000 C CNN
-F 2 "Connector_Molex:Molex_Mini-Fit_Jr_5566-20A_2x10_P4.20mm_Vertical" H 9850 1200 50  0001 C CNN
-F 3 "https://web.aub.edu.lb/pub/docs/atx_201.pdf#page=20" H 10950 750 50  0001 C CNN
-	1    9850 1300
-	1    0    0    -1
-$EndComp
-NoConn ~ 10350 1300
-Wire Wire Line
-	10350 1200 10450 1200
-Wire Wire Line
-	10450 1200 10450 1300
 Text GLabel 850  1700 0    50   Input ~ 0
 RES_IN
@@
 $EndComp
 Wire Wire Line
-	10350 1100 10550 1100
-Wire Wire Line
-	10450 1300 10550 1300
-Wire Wire Line
-	9850 1900 9850 2000
-Wire Wire Line
 	1350 4300 2650 4300
 Wire Wire Line
@@
 F1 "disk.sch" 50
 $EndSheet
-Text GLabel 8800 1800 1    50   Input ~ 0
-A0
-Text GLabel 8700 1800 1    50   Input ~ 0
-A1
 Text GLabel 8600 1800 1    50   Input ~ 0
 A2
@@
 Wire Wire Line
 	14950 1800 14600 1800
-NoConn ~ 10350 1700
 Wire Wire Line
 	15450 1900 15650 1900
@@
 Wire Wire Line
 	14950 2300 14600 2300
-Wire Wire Line
-	10350 1400 10600 1400
-Wire Wire Line
-	10600 1400 10600 1500
-Wire Wire Line
-	10600 1500 10650 1500
-$Comp
-L power:+3.3V #PWR0119
-U 1 1 631AAD95
-P 10650 1500
-F 0 "#PWR0119" H 10650 1350 50  0001 C CNN
-F 1 "+3.3V" V 10665 1628 50  0000 L CNN
-F 2 "" H 10650 1500 50  0001 C CNN
-F 3 "" H 10650 1500 50  0001 C CNN
-	1    10650 1500
-	0    1    1    0
-$EndComp
+$Comp
+L Connector:Screw_Terminal_01x03 J1
+U 1 1 62C98C2C
+P 11700 800
+F 0 "J1" H 11780 842 50  0000 L CNN
+F 1 "Screw_Terminal_01x03" H 11780 751 50  0000 L CNN
+F 2 "TerminalBlock_RND:TerminalBlock_RND_205-00277_1x03_P5.00mm_Vertical" H 11700 800 50  0001 C CNN
+F 3 "~" H 11700 800 50  0001 C CNN
+	1    11700 800
+	1    0    0    -1
+$EndComp
+Text GLabel 8700 1800 1    50   Input ~ 0
+A1
+Text GLabel 8800 1800 1    50   Input ~ 0
+A0
+$Comp
+L power:GND #PWR0119
+U 1 1 62D2FE61
+P 12150 1750
+F 0 "#PWR0119" H 12150 1500 50  0001 C CNN
+F 1 "GND" H 12155 1577 50  0000 C CNN
+F 2 "" H 12150 1750 50  0001 C CNN
+F 3 "" H 12150 1750 50  0001 C CNN
+	1    12150 1750
+	1    0    0    -1
+$EndComp
+Wire Wire Line
+	12150 1650 12150 1750
+Wire Wire Line
+	11050 800  11500 800
+Wire Wire Line
+	11350 700  11450 700
+Wire Wire Line
+	11350 900  11400 900
+$Comp
+L power:PWR_FLAG #FLG0101
+U 1 1 62DD2FC6
+P 11450 700
+F 0 "#FLG0101" H 11450 775 50  0001 C CNN
+F 1 "PWR_FLAG" H 11450 873 50  0000 C CNN
+F 2 "" H 11450 700 50  0001 C CNN
+F 3 "~" H 11450 700 50  0001 C CNN
+	1    11450 700
+	1    0    0    -1
+$EndComp
+Connection ~ 11450 700
+Wire Wire Line
+	11450 700  11500 700
+$Comp
+L power:PWR_FLAG #FLG0102
+U 1 1 62DD3384
+P 11400 900
+F 0 "#FLG0102" H 11400 975 50  0001 C CNN
+F 1 "PWR_FLAG" H 11400 1073 50  0000 C CNN
+F 2 "" H 11400 900 50  0001 C CNN
+F 3 "~" H 11400 900 50  0001 C CNN
+	1    11400 900
+	-1   0    0    1
+$EndComp
+Connection ~ 11400 900
+Wire Wire Line
+	11400 900  11500 900
 $EndSCHEMATC
